Commit message: feat: Update Go2W robot visuals with DAE files and add license

File: legged_gym/resources/robots/go2w/urdf/go2w.urdf (robot description, URDF)
Before this commit: robot go2w_description, 33 links, 32 joints
Links:
- link FL_calf: geometry collision cylinder length=0.12 radius=0.012; visual mesh filename=../meshes/calf.dae
- link FR_calf: geometry collision cylinder length=0.12 radius=0.013; visual mesh filename=../meshes/calf_mirror.dae
- link RL_calf: geometry collision cylinder length=0.12 radius=0.013; visual mesh filename=../meshes/calf.dae
- link RR_calf: geometry collision cylinder length=0.12 radius=0.013; visual mesh filename=../meshes/calf_mirror.dae

Commit message: Refactor sim2sim codebase for improved functionality and structure
- Updated model path in config.py to point directly to the new XML file.
- Enhanced command handling in controller.py to support scheduling of commands with validation.
- Removed doctor.py as it is no longer needed.
- Added export_checkpoint.py to facilitate exporting the TrackinBIT checkpoint without Isaac Gym.
- Refined policy.py to align with the new 53- and 57-dimensional Go2W policy layouts.
- Cleaned up requirements files by removing unnecessary dependencies.
- Modified run.py to enforce required policy argument and improved model validation.
- Updated simulator.py to include better handling of policy targets and simulation timing.
- Removed outdated test_contract.py to streamline testing efforts.

File: legged_gym/resources/robots/go2w/urdf/go2w.urdf (robot description, URDF)
Before this commit: robot go2w_description, 33 links, 32 joints
Links:
- link FL_calf: geometry collision cylinder length=0.12 radius=0.012; visual mesh filename=../meshes/calf.stl
- link FL_foot: geometry collision cylinder length=0.045 radius=0.086; visual mesh filename=../meshes/left_wheel.dae
- link FR_calf: geometry collision cylinder length=0.12 radius=0.013; visual mesh filename=../meshes/calf_mirror.stl
- link FR_foot: geometry collision cylinder length=0.045 radius=0.086; visual mesh filename=../meshes/right_wheel.dae
- link RL_calf: geometry collision cylinder length=0.12 radius=0.013; visual mesh filename=../meshes/calf.stl
- link RL_foot: geometry collision cylinder length=0.045 radius=0.086; visual mesh filename=../meshes/left_wheel.dae
- link RR_calf: geometry collision cylinder length=0.12 radius=0.013; visual mesh filename=../meshes/calf_mirror.stl
- link RR_foot: geometry collision cylinder length=0.045 radius=0.086; visual mesh filename=../meshes/right_wheel.dae

Commit message: Update URDF and XML configurations for GO2W robot
- Changed mesh file format from STL to DAE for calf and calf_mirror models.
- Modified foot joints from 'continuous' to 'revolute' type for better articulation.
- Updated joint limits to allow for a wider range of motion by setting lower and upper limits to -999999 and 999999 respectively.

File: legged_gym/resources/robots/go2w/urdf/go2w.urdf (robot description, URDF)
Before this commit: robot go2w_description, 33 links, 32 joints
Links:
- link FL_calf: geometry collision cylinder length=0.12 radius=0.012; visual mesh filename=../meshes/calf.dae
- link FR_calf: geometry collision cylinder length=0.12 radius=0.013; visual mesh filename=../meshes/calf_mirror.dae
- link RL_calf: geometry collision cylinder length=0.12 radius=0.013; visual mesh filename=../meshes/calf.dae
- link RR_calf: geometry collision cylinder length=0.12 radius=0.013; visual mesh filename=../meshes/calf_mirror.dae
Joints:
- joint FL_foot_joint: limit effort=23.7 velocity=30.1 -> lower=-999999 upper=999999 effort=23.7 velocity=30.1; type continuous -> revolute
- joint FR_foot_joint: limit effort=23.7 velocity=30.1 -> lower=-999999 upper=999999 effort=23.7 velocity=30.1; type continuous -> revolute
- joint RL_foot_joint: limit effort=23.7 velocity=30.1 -> lower=-999999 upper=999999 effort=23.7 velocity=30.1; type continuous -> revolute
- joint RR_foot_joint: limit effort=23.7 velocity=30.1 -> lower=-999999 upper=999999 effort=23.7 velocity=30.1; type continuous -> revolute
